File: placa_base/Placa_base_2layers/Placa_base.kicad_sch (KiCad schematic)
At the start: 50 parts, among them J1 Conn_01x16 Hembra, J10 Barrel_Jack 9V, J11 Conn_01x04 Macho, J2 Conn_01x16 Hembra, J3 Conn_01x03 Macho, J4 Conn_01x03 Macho, J5 Conn_01x05 Hembra, J6 Conn_01x03 Macho, J7 Conn_01x03 Macho, J8 Conn_01x04 Hembra, J9 Screw_Terminal_01x02, Q1 BD139, Q2 BC337, SW1 SW_Push, SW2 SW_Push, SW3 SW_Push, SW4 SW_Push, SW5 SW_SPST

Commit message: Please enter the commit message for your changes. Lines starting  with '#' will be ignored, and an empty message aborts the commit.
 On branch master
 Your branch is up to date with 'Entrenador2023/master'.

 Changes to be committed:
	modified:   desktop.ini
	deleted:    placa_base/Placa_base_2layers/#auto_saved_files#
	modified:   placa_base/Placa_base_2layers/Documentacion/datasheets/desktop.ini
	modified:   placa_base/Placa_base_2layers/Documentacion/desktop.ini
	deleted:    placa_base/Placa_base_2layers/Placa_base-backups/Placa_base-2023-01-19_191132.zip
	deleted:    placa_base/Placa_base_2layers/Placa_base-backups/Placa_base-2023-01-19_195627.zip
	deleted:    placa_base/Placa_base_2layers/Placa_base-backups/Placa_base-2023-01-19_215532.zip
	deleted:    placa_base/Placa_base_2layers/Placa_base-backups/Placa_base-2023-05-10_143256.zip
	deleted:    placa_base/Placa_base_2layers/Placa_base-backups/Placa_base-2023-05-10_144330.zip
	new file:   placa_base/Placa_base_2layers/Placa_base-backups/Placa_base-2023-05-10_162002.zip
	new file:   placa_base/Placa_base_2layers/Placa_base-backups/Placa_base-2023-05-11_185711.zip
	new file:   placa_base/Placa_base_2layers/Placa_base-backups/Placa_base-2023-05-11_194102.zip
	new file:   placa_base/Placa_base_2layers/Placa_base-backups/Placa_base-2023-05-11_201145.zip
	new file:   placa_base/Placa_base_2layers/Placa_base-backups/Placa_base-2023-05-12_190805.zip
	new file:   placa_base/Placa_base_2layers/Placa_base-backups/Placa_base-2023-05-15_084500.zip
	modified:   placa_base/Placa_base_2layers/Placa_base-backups/desktop.ini
	modified:   placa_base/Placa_base_2layers/Placa_base.kicad_pcb
	modified:   placa_base/Placa_base_2layers/Placa_base.kicad_prl
	modified:   placa_base/Placa_base_2layers/Placa_base.kicad_sch
	deleted:    placa_base/Placa_base_2layers/_autosave-Placa_base.kicad_sch
	modified:   placa_base/Placa_base_2layers/desktop.ini
	modified:   placa_base/Placa_base_2layers/fabrication/desktop.ini
	modified:   placa_base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
Parts:
- C6: footprint Capacitor_THT:CP_Radial_D7.5mm_P2.50mm -> Capacitor_THT:CP_Radial_D8.0mm_P3.50mm
Changed lines of the file:
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@@
       (effects (font (size 1.27 1.27)) (justify left))
     )
-    (property "Footprint" "Capacitor_THT:CP_Radial_D7.5mm_P2.50mm" (at 267.6652 107.95 0)
+    (property "Footprint" "Capacitor_THT:CP_Radial_D8.0mm_P3.50mm" (at 267.6652 107.95 0)
       (effects (font (size 1.27 1.27)) hide)
     )
